Commit message: feat(obstacle_avoider): automatically detect obstacles around to move

File: config/my_robot.urdf (robot description, URDF)
Before this commit: robot robot model, 4 links, 3 joints
Joints:
- joint base_footprint_to_base_link: limit lower=-100 upper=100 effort=100 velocity=100 -> (none)
- joint base_to_left_wheel: axis 0 1 0 -> (none)
- joint base_to_right_wheel: axis 0 1 0 -> (none)
